Commit message: update the urdf

File: src/Anton_description/urdf/Anton_description.urdf (robot description, URDF)
Before this commit: robot Anton, 3 links, 2 joints
Links:
- added link laser_link; visual cylinder length=${laser_length} radius=${laser_radius}
Joints:
- added joint laser_joint: type fixed, parent base_link, child laser_link

Commit message: let the robots move manually
finished tasks of US2 TASK 25. 26, 27, 28

File: src/Anton_description/urdf/Anton_description.urdf (robot description, URDF)
Before this commit: robot Anton, 5 links, 4 joints
Links:
- removed link laser_link
- link base_link: geometry collision box size=${base_length} ${base_width} ${base_height}; visual box size=${base_length} ${base_width} ${base_height}
- link front_caster: geometry collision sphere radius=${(wheel_radius+wheel_zoff-(base_height/2))}; visual sphere radius=${(wheel_radius+wheel_zoff-(base_height/2))}
Joints:
- removed joint laser_joint
