Commit message: [US90 Task108] make the scaled rover movable

File: src/Anton_description/urdf/roverTest.urdf (robot description, URDF)
Before this commit: robot Anton, 7 links, 6 joints
Links:
- link camera_link: geometry collision box size=0.015 0.130 0.022; visual box size=0.015 0.130 0.022
- link imu_link: geometry collision box size=0.1 0.1 0.1; visual box size=0.1 0.1 0.1
Joints:
- joint camera_joint: origin xyz=0.215 0 0.05 rpy=0 0 0 -> xyz=${base_length / 2} 0 0.05 rpy=0 0 0
- joint lidar_joint: origin xyz=0 0 0.12 rpy=0 0 0 -> xyz=0 0 ${base_height / 2 + 0.02} rpy=0 0 0
