Commit message: [US127 Task???] provided more config files for parts of rover

File: src/Anton_description/urdf/Anton.urdf (robot description, URDF)
Before this commit: robot Anton, 8 links, 7 joints
Links:
- link base_link: geometry collision box size=0.42 0.31 0.18; visual box size=0.42 0.31 0.18
Joints:
- joint base_joint: child base_link -> base_footprint; parent base_footprint -> base_link
- joint camera_joint: origin xyz=0.165 0 -0.035 rpy=0 0 0 -> xyz=0.165 0 0.05 rpy=0 0 0
- joint caster_joint: origin xyz=-0.052 0 -0.055 rpy=0 0 0 -> xyz=0.14 0 -0.09 rpy=0 0 0; type continuous -> fixed

File: src/Anton_description/urdf/Anton.xacro (robot description, xacro)
@@ -1,5 +1,7 @@
 <?xml version="1.0"?>
 <robot name="Anton" xmlns:xacro="http://www.ros.org/wiki/xacro">
-  <xacro:include filename="./dimensions.xacro"/>
+  <xacro:include filename="./chasis_dimension_1.xacro"/>
+  <xacro:include filename="./wheels_dimension_1.xacro"/>
+  <xacro:include filename="./caster_dimension_1.xacro"/>
   <xacro:include filename="./chasis.xacro"/>
   <xacro:include filename="./wheels.xacro"/>

File: src/Anton_description/urdf/camera.xacro (robot description, xacro)
@@ -6,5 +6,5 @@
     <xacro:property name="camera_origin_x" value="0.165"/>
     <xacro:property name="camera_origin_y" value="0"/>
-    <xacro:property name="camera_origin_z" value="-0.035"/>
+    <xacro:property name="camera_origin_z" value="0.05"/>
     <link name="camera_link">
         <visual>

File: src/Anton_description/urdf/caster.xacro (robot description, xacro)
@@ -1,30 +1,30 @@
 <?xml version="1.0"?>
 <robot name="Anton" xmlns:xacro="http://www.ros.org/wiki/xacro">
-<xacro:macro name="sphere_inertia" params="m r">
-  <inertial>
-    <mass value="${m}"/>
-    <inertia ixx="${2.0*m*(r*r)/5.0}" ixy="0.0" ixz="0.0" iyy="${2.0*m*(r*r)/5.0}" iyz="0.0" izz="${2.0*m*(r*r)/5.0}"/>
-  </inertial>
-</xacro:macro>
-<link name="front_caster">
-  <visual>
-    <origin xyz="0 0 0" rpy="0 0 0"/>
-    <geometry>
-      <sphere radius="${caster_wheel_radius}"/>
-    </geometry>
-  </visual>
-  <collision>
-    <origin xyz="0 0 0" rpy="0 0 0"/>
-    <geometry>
-      <sphere radius="${caster_wheel_radius}"/>
-    </geometry>
-  </collision>
-  <xacro:sphere_inertia m="5" r="${caster_wheel_radius}"/>
-</link>
-<joint name="caster_joint" type="continuous">
-  <axis xyz="0 1 0" rpy="0 0 0" />
-  <parent link="base_link"/>
-  <child link="front_caster"/>
-  <origin xyz="${caster_wheel_joint_offset} 0 -${caster_wheel_radius+0.005}" rpy="0 0 0"/>
-</joint>
+  <xacro:macro name="sphere_inertia" params="m r">
+    <inertial>
+      <mass value="${m}"/>
+      <inertia ixx="${2.0*m*(r*r)/5.0}" ixy="0.0" ixz="0.0" iyy="${2.0*m*(r*r)/5.0}" iyz="0.0" izz="${2.0*m*(r*r)/5.0}"/>
+    </inertial>
+  </xacro:macro>
+  <link name="front_caster">
+    <visual>
+      <origin xyz="0 0 0" rpy="0 0 0"/>
+      <geometry>
+        <sphere radius="${caster_wheel_radius}"/>
+      </geometry>
+    </visual>
+    <collision>
+      <origin xyz="0 0 0" rpy="0 0 0"/>
+      <geometry>
+        <sphere radius="${caster_wheel_radius}"/>
+      </geometry>
+    </collision>
+    <xacro:sphere_inertia m="5" r="${caster_wheel_radius}"/>
+  </link>
+  <joint name="caster_joint" type="fixed">
+    <axis xyz="0 1 0" rpy="0 0 0" />
+    <parent link="base_link"/>
+    <child link="front_caster"/>
+    <origin xyz="${caster_wheel_joint_offset} 0 -${base_height/2}" rpy="0 0 0"/>
+  </joint>
 </robot>

File: src/Anton_description/urdf/chasis.xacro (robot description, xacro)
@@ -1,36 +1,36 @@
 <?xml version="1.0"?>
 <robot name="Anton" xmlns:xacro="http://www.ros.org/wiki/xacro">
-<xacro:macro name="box_inertia" params="m w h d">
-  <inertial>
-    <mass value="${m}"/>
-    <inertia ixx="${m / 12.0 * (d*d + h*h)}" ixy="0.0" ixz="0.0" iyy="${m / 12.0 * (w*w + h*h)}" iyz="0.0" izz="${m / 12.0 * (w*w + d*d)}"/>
-  </inertial>
-</xacro:macro>
-<link name="base_footprint">
-  <xacro:box_inertia m="20" w="0.001" h="0.001" d="0.001"/>
-  <visual>
-    <origin xyz="0 0 0" rpy="0 0 0" />
-    <geometry>
-       <box size="0.001 0.001 0.001" />
-    </geometry>
-  </visual>
-</link>
-<link name="base_link">
-  <xacro:box_inertia m="10" w="${base_length}" h="${base_width}" d="0.01"/>
-  <visual>
-    <geometry>
-      <box size="${base_length} ${base_width} 0.01"/>
-    </geometry>
-  </visual>
-  <collision>
-    <geometry>
-      <box size="${base_length} ${base_width} 0.01"/>
-    </geometry>
-  </collision>
-</link>
-<joint name="base_joint" type="fixed">
-  <origin xyz="0 0 ${wheel_radius + 0.005}" rpy="0 0 0" />
-  <parent link="base_footprint"/>
-  <child link="base_link" />
-</joint>
+  <xacro:macro name="box_inertia" params="m w h d">
+    <inertial>
+      <mass value="${m}"/>
+      <inertia ixx="${m / 12.0 * (d*d + h*h)}" ixy="0.0" ixz="0.0" iyy="${m / 12.0 * (w*w + h*h)}" iyz="0.0" izz="${m / 12.0 * (w*w + d*d)}"/>
+    </inertial>
+  </xacro:macro>
+  <link name="base_footprint">
+    <xacro:box_inertia m="20" w="0.001" h="0.001" d="0.001"/>
+    <visual>
+      <origin xyz="0 0 0" rpy="0 0 0" />
+      <geometry>
+         <box size="0.001 0.001 0.001" />
+      </geometry>
+    </visual>
+  </link>
+  <link name="base_link">
+    <xacro:box_inertia m="10" w="${base_length}" h="${base_width}" d="${base_height}"/>
+    <visual>
+      <geometry>
+        <box size="${base_length} ${base_width} ${base_height}"/>
+      </geometry>
+    </visual>
+    <collision>
+      <geometry>
+        <box size="${base_length} ${base_width} ${base_height}"/>
+      </geometry>
+    </collision>
+  </link>
+  <joint name="base_joint" type="fixed">
+    <origin xyz="0 0 ${wheel_radius + 0.005}" rpy="0 0 0" />
+    <parent link="base_link"/>
+    <child link="base_footprint" />
+  </joint>
 </robot>

File: src/Anton_description/urdf/dimensions.xacro (robot description, xacro)
@@ -17,4 +17,4 @@
   <xacro:property name="caster_wheel_radius" value="${wheel_radius/2}"/>
   <xacro:property name="caster_wheel_mass" value="0.001"/>
-  <xacro:property name="caster_wheel_joint_offset" value="-0.052"/>
+  <xacro:property name="caster_wheel_joint_offset" value="0.14"/>
 </robot>

Commit message: [US129 TASK150] edited  multiple config files for user to choose

File: src/Anton_description/urdf/Anton.urdf (robot description, URDF)
Before this commit: robot Anton, 8 links, 7 joints
Links:
- added link imu_link, mass 0.1; collision box size=0.1 0.1 0.1; visual box size=0.1 0.1 0.1
- link base_footprint: mass 20 -> None; geometry 
- link base_link: mass 10 -> 30; geometry collision box size=0.53 0.31 0.1; visual box size=0.53 0.31 0.1
- link camera_link: mass 0.2 -> 0.035; geometry collision box size=0.015 0.13 0.022; visual box size=0.015 0.13 0.022
- link drivewhl_l_link: geometry collision cylinder length=0.06 radius=0.15; visual cylinder length=0.06 radius=0.15
- link drivewhl_r_link: geometry collision cylinder length=0.06 radius=0.15; visual cylinder length=0.06 radius=0.15
- link front_caster: geometry collision sphere radius=0.09999999999999999; visual sphere radius=0.09999999999999999
Joints:
- added joint imu_joint: type fixed, parent base_link, child imu_link, origin xyz=0 0 0.01 rpy=0 0 0
- joint base_joint: origin xyz=0 0 0.10500000000000001 rpy=0 0 0 -> xyz=0 0 -0.2 rpy=0 0 0
- joint camera_joint: origin xyz=0.165 0 0.05 rpy=0 0 0 -> xyz=0.265 0 0.05 rpy=0 0 0
- joint caster_joint: origin xyz=0.14 0 -0.09 rpy=0 0 0 -> xyz=0.17666666666666667 0 -0.05 rpy=0 0 0

File: src/Anton_description/urdf/Anton.xacro (robot description, xacro)
@@ -7,4 +7,5 @@
   <xacro:include filename="./wheels.xacro"/>
   <xacro:include filename="./caster.xacro"/>
+  <xacro:include filename="./imu.xacro"/>
   <xacro:include filename="./laser.xacro"/>
   <xacro:include filename="./camera.xacro"/>

File: src/Anton_description/urdf/DDCplugin.xacro (robot description, xacro)
@@ -10,6 +10,6 @@
       <right_joint>drivewhl_r_joint</right_joint>
       <!-- kinematics -->
-      <wheel_separation>0.4</wheel_separation>
-      <wheel_diameter>0.2</wheel_diameter>
+      <wheel_separation>${wheel_separation}</wheel_separation>
+      <wheel_diameter>${wheel_radius*2}</wheel_diameter>
       <!-- limits -->
       <max_wheel_torque>20</max_wheel_torque>

File: src/Anton_description/urdf/camera.xacro (robot description, xacro)
@@ -1,10 +1,10 @@
 <?xml version="1.0"?>
 <robot name="Anton" xmlns:xacro="http://www.ros.org/wiki/xacro">
-    <xacro:property name="camera_size_x" value="0.03"/>
-    <xacro:property name="camera_size_y" value="0.03"/>
-    <xacro:property name="camera_size_z" value="0.04"/>
-    <xacro:property name="camera_origin_x" value="0.165"/>
+    <xacro:property name="camera_size_x" value="0.015"/>
+    <xacro:property name="camera_size_y" value="0.13"/>
+    <xacro:property name="camera_size_z" value="0.022"/>
+    <xacro:property name="camera_origin_x" value="${base_length/2}"/>
     <xacro:property name="camera_origin_y" value="0"/>
-    <xacro:property name="camera_origin_z" value="0.05"/>
+    <xacro:property name="camera_origin_z" value="${base_height/2}"/>
     <link name="camera_link">
         <visual>
@@ -19,5 +19,5 @@
             </geometry>
         </collision>
-        <xacro:box_inertia m="0.2" w="${camera_size_x}" h="${camera_size_y}" d="${camera_size_z}"/>
+        <xacro:box_inertia m="0.035" w="${camera_size_x}" h="${camera_size_y}" d="${camera_size_z}"/>
     </link>
     <joint name="camera_joint" type="fixed">

File: src/Anton_description/urdf/caster_dimension_2.xacro (robot description, xacro)
@@ -3,4 +3,4 @@
   <xacro:property name="caster_wheel_radius" value="${wheel_radius/3}"/>
   <xacro:property name="caster_wheel_mass" value="0.001"/>
-  <xacro:property name="caster_wheel_joint_offset" value="${base_length/3}"/>
+  <xacro:property name="caster_wheel_joint_offset" value="${base_length/2}"/>
 </robot>

File: src/Anton_description/urdf/chasis.xacro (robot description, xacro)
@@ -7,15 +7,7 @@
     </inertial>
   </xacro:macro>
-  <link name="base_footprint">
-    <xacro:box_inertia m="20" w="0.001" h="0.001" d="0.001"/>
-    <visual>
-      <origin xyz="0 0 0" rpy="0 0 0" />
-      <geometry>
-         <box size="0.001 0.001 0.001" />
-      </geometry>
-    </visual>
-  </link>
+  <link name="base_footprint"/>
   <link name="base_link">
-    <xacro:box_inertia m="10" w="${base_length}" h="${base_width}" d="${base_height}"/>
+    <xacro:box_inertia m="30" w="${base_length}" h="${base_width}" d="${base_height}"/>
     <visual>
       <geometry>
@@ -30,5 +22,5 @@
   </link>
   <joint name="base_joint" type="fixed">
-    <origin xyz="0 0 ${wheel_radius + 0.005}" rpy="0 0 0" />
+    <origin xyz="0 0 ${-(wheel_radius+wheel_zoff)}" rpy="0 0 0" />
     <parent link="base_link"/>
     <child link="base_footprint" />

File: src/Anton_description/urdf/chasis_dimension_2.xacro (robot description, xacro)
@@ -1,5 +1,5 @@
 <?xml version="1.0"?>
 <robot name="Anton" xmlns:xacro="http://www.ros.org/wiki/xacro">
-  <xacro:property name="base_width" value="0.15"/>
+  <xacro:property name="base_width" value="0.31"/>
   <xacro:property name="base_length" value="0.2"/>
   <xacro:property name="base_height" value="0.1"/>

File: src/Anton_description/urdf/chasis_dimension_3.xacro (robot description, xacro)
@@ -1,5 +1,5 @@
 <?xml version="1.0"?>
 <robot name="Anton" xmlns:xacro="http://www.ros.org/wiki/xacro">
-  <xacro:property name="base_width" value="0.45"/>
+  <xacro:property name="base_width" value="0.31"/>
   <xacro:property name="base_length" value="0.53"/>
   <xacro:property name="base_height" value="0.1"/>

File: src/Anton_description/urdf/imu.xacro (robot description, xacro)
@@ -1,10 +1,10 @@
 <?xml version="1.0"?>
 <robot name="Anton" xmlns:xacro="http://www.ros.org/wiki/xacro">
-  <xacro:property name="IMUsizeX" value="0.01"/>
-  <xacro:property name="IMUsizeY" value="0.01"/>
-  <xacro:property name="IMUsizeZ" value="0.01"/>
+  <xacro:property name="IMUsizeX" value="0.1"/>
+  <xacro:property name="IMUsizeY" value="0.1"/>
+  <xacro:property name="IMUsizeZ" value="0.1"/>
   <xacro:property name="IMUoriginX" value="0"/>
   <xacro:property name="IMUoriginY" value="0"/>
-  <xacro:property name="IMUoriginZ" value="0.015"/>
+  <xacro:property name="IMUoriginZ" value="0.01"/>
   <link name="imu_link">
     <visual>
@@ -19,10 +19,10 @@
       </geometry>
     </collision>
-    <xacro:box_inertia m="0.2" w="${IMUsizeX}" h="${IMUsizeY}" d="${IMUsizeZ}"/>
+    <xacro:box_inertia m="0.1" w="${IMUsizeX}" h="${IMUsizeY}" d="${IMUsizeZ}"/>
   </link>
   <joint name="imu_joint" type="fixed">
     <origin xyz="${IMUoriginX} ${IMUoriginY} ${IMUoriginZ}" rpy="0 0 0" />
     <parent link="base_link"/>
-    <child link= imu_link" />
+    <child link="imu_link"/>
   </joint>
 </robot>

File: src/Anton_description/urdf/wheels_dimension_1.xacro (robot description, xacro)
@@ -2,5 +2,5 @@
 <robot name="Anton" xmlns:xacro="http://www.ros.org/wiki/xacro">
   <xacro:property name="base_wheel_gap" value="0.007"/>
-	<xacro:property name="wheel_separation" value="0.15"/>
+	<xacro:property name="wheel_separation" value="0.4"/>
   <xacro:property name="wheel_joint_offset" value="0.02"/>
   <xacro:property name="wheel_radius" value="0.10"/>

Commit message: [US129 TASK151] updated the position of the lidar to avoid ray blocking by rover body

File: src/Anton_description/urdf/Anton.urdf (robot description, URDF)
Before this commit: robot Anton, 9 links, 8 joints
Links:
- link base_link: geometry collision box size=0.42 0.31 0.18; visual box size=0.42 0.31 0.18
- link drivewhl_l_link: geometry collision cylinder length=0.04 radius=0.1; visual cylinder length=0.04 radius=0.1
- link drivewhl_r_link: geometry collision cylinder length=0.04 radius=0.1; visual cylinder length=0.04 radius=0.1
- link front_caster: geometry collision sphere radius=0.05; visual sphere radius=0.05
Joints:
- joint base_joint: origin xyz=0 0 -0.2 rpy=0 0 0 -> xyz=0 0 -0.15000000000000002 rpy=0 0 0
- joint camera_joint: origin xyz=0.265 0 0.05 rpy=0 0 0 -> xyz=0.21 0 0.09 rpy=0 0 0
- joint caster_joint: origin xyz=0.17666666666666667 0 -0.05 rpy=0 0 0 -> xyz=0.13999999999999999 0 -0.09 rpy=0 0 0
- joint lidar_joint: origin xyz=0 0 0.12 rpy=0 0 0 -> xyz=0 0 0.27 rpy=0 0 0

File: src/Anton_description/urdf/laser.xacro (robot description, xacro)
@@ -23,5 +23,5 @@
     <parent link="base_link"/>
     <child link="lidar_link"/>
-    <origin xyz="0 0 0.12" rpy="0 0 0"/>
+    <origin xyz="0 0 ${base_height*3/2}" rpy="0 0 0"/>
   </joint>
 </robot>
