Commit message: [US127 TASK142] xacro files are able to be translated to urdf

File: src/Anton_description/urdf/xacro/Anton.xacro (robot description, xacro)
@@ -1,10 +1,10 @@
 <?xml version="1.0"?>
 <robot name="Anton" xmlns:xacro="http://www.ros.org/wiki/xacro">
-  <xacro:include filename="$(find Anton_description)/urdf/xacro/dimensions.xacro"/>
-  <xacro:include filename="$(find Anton_description)/urdf/xacro/chasis.xacro"/>
-  <xacro:include filename="$(find Anton_description)/urdf/xacro/wheels.xacro"/>
-  <xacro:include filename="$(find Anton_description)/urdf/xacro/caster.xacro"/>
-  <xacro:include filename="$(find Anton_description)/urdf/xacro/laser.xacro"/>
-  <xacro:include filename="$(find Anton_description)/urdf/xacro/camera.xacro"/>
-  <xacro:include filename="$(find Anton_description)/urdf/xacro/AntonPlugins.xacro"/>
+  <xacro:include filename="./dimensions.xacro"/>
+  <xacro:include filename="./chasis.xacro"/>
+  <xacro:include filename="./wheels.xacro"/>
+  <xacro:include filename="./caster.xacro"/>
+  <xacro:include filename="./laser.xacro"/>
+  <xacro:include filename="./camera.xacro"/>
+  <xacro:include filename="./AntonPlugins.xacro"/>
 </robot>

File: src/Anton_description/urdf/xacro/AntonPlugins.xacro (robot description, xacro)
@@ -1,8 +1,8 @@
 <?xml version="1.0" ?>
 <robot name="Anton" xmlns:xacro="https://www.ros.org/wiki/xacro" >
-  <xacro:include filename="$(find Anton_description)/urdf/xacro/visuals.xacro"/>
-  <xacro:include filename="$(find Anton_description)/urdf/xacro/DDCplugin.xacro"/>
-  <xacro:include filename="$(find Anton_description)/urdf/xacro/laserPlugin.xacro"/>
-  <xacro:include filename="$(find Anton_description)/urdf/xacro/cameraPplugin.xacro"/>
-  <xacro:include filename="$(find Anton_description)/urdf/xacro/imuPlugin.xacro"/>
+  <xacro:include filename="./visuals.xacro"/>
+  <xacro:include filename="./DDCplugin.xacro"/>
+  <xacro:include filename="./laserPlugin.xacro"/>
+  <xacro:include filename="./cameraPlugin.xacro"/>
+  <xacro:include filename="./imuPlugin.xacro"/>
 </robot>

File: src/Anton_description/urdf/xacro/camera.xacro (robot description, xacro)
@@ -24,5 +24,5 @@
         <origin xyz="${camera_origin_x} ${camera_origin_y} ${camera_origin_z}" rpy="0 0 0" />
         <parent link="base_link"/>
-            <child link= “camera_link" />
+            <child link="camera_link" />
     </joint>
 </robot>

File: src/Anton_description/urdf/xacro/cameraPlugin.xacro (robot description, xacro)
@@ -9,5 +9,5 @@
          horizontal_fov> -->
         <horizontal_fov>1.57</horizontal_fov>
-        <!— ~90 degrees -->
+        <!-- ~90 degrees -->
         <image>
           <width>800</width>
@@ -34,9 +34,7 @@
           <alwaysOn>true</alwaysOn>
         <updateRate>0.0</updateRate>
-        <cameraName>ai_rover_remastered/camera1</
-         cameraName>
+        <cameraName>ai_rover_remastered/camera1</cameraName>
         <imageTopicName>image_raw</imageTopicName>
-        <cameraInfoTopicName>camera_info</
-         cameraInfoTopicName>
+        <cameraInfoTopicName>camera_info</cameraInfoTopicName>
         <frameName>camera_link</frameName>
         <hackBaseline>0.07</hackBaseline>
