Commit message: [US127 TASK143] updated the xacro files with our rviz config names

File: src/Anton_description/urdf/xacro/DDCplugin.xacro (robot description, xacro)
@@ -2,23 +2,23 @@
 <robot name="Anton" xmlns:xacro="https://www.ros.org/wiki/xacro" >
   <gazebo>
-    <plugin name="differential_drive_controller" filename="libgazebo_ros_diff_drive.so">
-      <alwaysOn>false</alwaysOn>
-      <legacyMode>false</legacyMode>
-      <updateRate>20</updateRate>
-      <leftJoint>left_wheel_joint</leftJoint>
-      <rightJoint>right_wheel_joint</rightJoint>
-      <wheelSeparation> ${wheel_separation}
-      </wheelSeparation>
-      <wheelDiameter>${wheel_radius * 2}
-      </wheelDiameter>
-      <torque>20</torque>
-      <commandTopic>
-        /ai_rover_remastered/base_controller/cmd_vel
-      </commandTopic>
-      <odometryTopic>
-        /ai_rover_remastered/base_controller/odom
-      </odometryTopic>
-      <odometryFrame>odom</odometryFrame>
-      <robotBaseFrame>base_footprint</robotBaseFrame>
+    <plugin name='diff_drive' filename='libgazebo_ros_diff_drive.so'>
+      <ros>
+        <!-- <namespace>/demo</namespace> -->
+      </ros>
+      <!-- wheels -->
+      <left_joint>drivewhl_l_joint</left_joint>
+      <right_joint>drivewhl_r_joint</right_joint>
+      <!-- kinematics -->
+      <wheel_separation>0.4</wheel_separation>
+      <wheel_diameter>0.2</wheel_diameter>
+      <!-- limits -->
+      <max_wheel_torque>20</max_wheel_torque>
+      <max_wheel_acceleration>1.0</max_wheel_acceleration>
+      <!-- output -->
+      <publish_odom>true</publish_odom>
+      <publish_odom_tf>false</publish_odom_tf>
+      <publish_wheel_tf>true</publish_wheel_tf>
+      <odometry_frame>odom</odometry_frame>
+      <robot_base_frame>base_link</robot_base_frame>
     </plugin>
   </gazebo>

File: src/Anton_description/urdf/xacro/camera.xacro (robot description, xacro)
@@ -24,5 +24,11 @@
         <origin xyz="${camera_origin_x} ${camera_origin_y} ${camera_origin_z}" rpy="0 0 0" />
         <parent link="base_link"/>
-            <child link="camera_link" />
+        <child link="camera_link" />
+    </joint>
+    <link name="camera_depth_frame"/>
+    <joint name="camera_depth_joint" type="fixed">
+        <origin xyz="0 0 0" rpy="${-pi/2} 0 ${-pi/2}"/>
+        <parent link="camera_link"/>
+        <child link="camera_depth_frame"/>
     </joint>
 </robot>

File: src/Anton_description/urdf/xacro/cameraPlugin.xacro (robot description, xacro)
@@ -2,46 +2,36 @@
 <robot name="Anton" xmlns:xacro="https://www.ros.org/wiki/xacro" >
   <gazebo reference="camera_link">
-    <sensor type="camera" name="camera1">
+    <sensor name="depth_camera" type="depth">
+      <visualize>true</visualize>
       <update_rate>30.0</update_rate>
-      <camera name="head">
-        <!--
-        <horizontal_fov>1.3962634</
-         horizontal_fov> -->
-        <horizontal_fov>1.57</horizontal_fov>
-        <!-- ~90 degrees -->
+      <camera name="camera">
+        <horizontal_fov>1.047198</horizontal_fov>
         <image>
-          <width>800</width>
-          <height>800</height>
+          <width>640</width>
+          <height>480</height>
           <format>R8G8B8</format>
         </image>
         <clip>
-          <near>0.02</near>
-          <far>300</far>
+          <near>0.05</near>
+          <far>3</far>
         </clip>
-        <noise>
-          <type>gaussian</type>
-          <!-- Noise is sampled independently per
-          pixel on each frame. Adding pixel's noise
-          value to each color
-          channels, which at that point lie in the
-          range [0,1]. -->
-          <mean>0.0</mean>
-          <stddev>0.007</stddev>
-        </noise>
       </camera>
-      <plugin name="camera_controller"
-       filename="libgazebo_ros_camera.so">
-          <alwaysOn>true</alwaysOn>
+      <plugin name="depth_camera_controller" filename="libgazebo_ros_camera.so">
+        <baseline>0.2</baseline>
+        <alwaysOn>true</alwaysOn>
         <updateRate>0.0</updateRate>
-        <cameraName>ai_rover_remastered/camera1</cameraName>
-        <imageTopicName>image_raw</imageTopicName>
-        <cameraInfoTopicName>camera_info</cameraInfoTopicName>
-        <frameName>camera_link</frameName>
-        <hackBaseline>0.07</hackBaseline>
-        <distortionK1>0.0</distortionK1>
-        <distortionK2>0.0</distortionK2>
-        <distortionK3>0.0</distortionK3>
-        <distortionT1>0.0</distortionT1>
-        <distortionT2>0.0</distortionT2>
+        <frame_name>camera_depth_frame</frame_name>
+        <pointCloudCutoff>0.5</pointCloudCutoff>
+        <pointCloudCutoffMax>3.0</pointCloudCutoffMax>
+        <distortionK1>0</distortionK1>
+        <distortionK2>0</distortionK2>
+        <distortionK3>0</distortionK3>
+        <distortionT1>0</distortionT1>
+        <distortionT2>0</distortionT2>
+        <CxPrime>0</CxPrime>
+        <Cx>0</Cx>
+        <Cy>0</Cy>
+        <focalLength>0</focalLength>
+        <hackBaseline>0</hackBaseline>
       </plugin>
     </sensor>

File: src/Anton_description/urdf/xacro/caster.xacro (robot description, xacro)
@@ -7,5 +7,5 @@
   </inertial>
 </xacro:macro>
-<link name="caster_wheel">
+<link name="front_caster">
   <visual>
     <origin xyz="0 0 0" rpy="0 0 0"/>
@@ -22,8 +22,8 @@
   <xacro:sphere_inertia m="5" r="${caster_wheel_radius}"/>
 </link>
-<joint name="caster_wheel_joint" type="continuous">
+<joint name="caster_joint" type="continuous">
   <axis xyz="0 1 0" rpy="0 0 0" />
   <parent link="base_link"/>
-  <child link="caster_wheel"/>
+  <child link="front_caster"/>
   <origin xyz="${caster_wheel_joint_offset} 0 -${caster_wheel_radius+0.005}" rpy="0 0 0"/>
 </joint>

File: src/Anton_description/urdf/xacro/chasis.xacro (robot description, xacro)
@@ -29,5 +29,5 @@
   </collision>
 </link>
-<joint name="base_link_joint" type="fixed">
+<joint name="base_joint" type="fixed">
   <origin xyz="0 0 ${wheel_radius + 0.005}" rpy="0 0 0" />
   <parent link="base_footprint"/>

File: src/Anton_description/urdf/xacro/dimensions.xacro (robot description, xacro)
@@ -1,10 +1,18 @@
 <?xml version="1.0"?>
 <robot name="Anton" xmlns:xacro="http://www.ros.org/wiki/xacro">
-  <xacro:property name="base_width" value="0.16"/>
-  <xacro:property name="base_length" value="0.16"/>
-  <xacro:property name="wheel_radius" value="0.035"/>
+  <!-- <xacro:property name="base_width" value="0.16"/>
+  <xacro:property name="base_length" value="0.16"/> -->
+  <!-- <xacro:property name="wheel_radius" value="0.035"/> -->
+  <xacro:property name="base_width" value="0.31"/>
+  <xacro:property name="base_length" value="0.42"/>
+  <xacro:property name="base_height" value="0.18"/>
   <xacro:property name="base_wheel_gap" value="0.007"/>
   <xacro:property name="wheel_separation" value="0.15"/>
   <xacro:property name="wheel_joint_offset" value="0.02"/>
+  <xacro:property name="wheel_radius" value="0.10"/>
+  <xacro:property name="wheel_width" value="0.04"/>
+  <xacro:property name="wheel_ygap" value="0.025"/>
+  <xacro:property name="wheel_zoff" value="0.05"/>
+  <xacro:property name="wheel_xoff" value="0.12"/>
   <xacro:property name="caster_wheel_radius" value="${wheel_radius/2}"/>
   <xacro:property name="caster_wheel_mass" value="0.001"/>

File: src/Anton_description/urdf/xacro/imu.xacro (robot description, xacro)
@@ -7,5 +7,5 @@
   <xacro:property name="IMUoriginY" value="0"/>
   <xacro:property name="IMUoriginZ" value="0.015"/>
-  <link name="IMU_link">
+  <link name="imu_link">
     <visual>
       <geometry>
@@ -21,8 +21,8 @@
     <xacro:box_inertia m="0.2" w="${IMUsizeX}" h="${IMUsizeY}" d="${IMUsizeZ}"/>
   </link>
-  <joint name="IMU_joint" type="fixed">
+  <joint name="imu_joint" type="fixed">
     <origin xyz="${IMUoriginX} ${IMUoriginY} ${IMUoriginZ}" rpy="0 0 0" />
     <parent link="base_link"/>
-    <child link= “IMU_link" />
+    <child link= imu_link" />
   </joint>
 </robot>

File: src/Anton_description/urdf/xacro/imuPlugin.xacro (robot description, xacro)
@@ -1,14 +1,71 @@
 <?xml version="1.0" ?>
 <robot name="Anton" xmlns:xacro="https://www.ros.org/wiki/xacro" >
-  <gazebo>
-    <plugin name="imu_plugin"
-      filename="libgazebo_ros_imu.so">
-      <alwaysOn>true</alwaysOn>
-      <bodyName>IMU_link</bodyName>
-      <topicName>imu</topicName>
-      <serviceName>imu_service</serviceName>
-      <gaussianNoise>0.0</gaussianNoise>
-      <updateRate>20.0</updateRate>
-    </plugin>
+  <gazebo reference="imu_link">
+    <sensor name="imu_sensor" type="imu">
+    <plugin filename="libgazebo_ros_imu_sensor.so" name="imu_plugin">
+        <ros>
+          <!-- <namespace>/demo</namespace> -->
+          <remapping>~/out:=imu</remapping>
+        </ros>
+        <initial_orientation_as_reference>false</initial_orientation_as_reference>
+      </plugin>
+      <always_on>true</always_on>
+      <update_rate>100</update_rate>
+      <visualize>true</visualize>
+      <imu>
+        <angular_velocity>
+          <x>
+            <noise type="gaussian">
+              <mean>0.0</mean>
+              <stddev>2e-4</stddev>
+              <bias_mean>0.0000075</bias_mean>
+              <bias_stddev>0.0000008</bias_stddev>
+            </noise>
+          </x>
+          <y>
+            <noise type="gaussian">
+              <mean>0.0</mean>
+              <stddev>2e-4</stddev>
+              <bias_mean>0.0000075</bias_mean>
+              <bias_stddev>0.0000008</bias_stddev>
+            </noise>
+          </y>
+          <z>
+            <noise type="gaussian">
+              <mean>0.0</mean>
+              <stddev>2e-4</stddev>
+              <bias_mean>0.0000075</bias_mean>
+              <bias_stddev>0.0000008</bias_stddev>
+            </noise>
+          </z>
+        </angular_velocity>
+        <linear_acceleration>
+          <x>
+            <noise type="gaussian">
+              <mean>0.0</mean>
+              <stddev>1.7e-2</stddev>
+              <bias_mean>0.1</bias_mean>
+              <bias_stddev>0.001</bias_stddev>
+            </noise>
+          </x>
+          <y>
+            <noise type="gaussian">
+              <mean>0.0</mean>
+              <stddev>1.7e-2</stddev>
+              <bias_mean>0.1</bias_mean>
+              <bias_stddev>0.001</bias_stddev>
+            </noise>
+          </y>
+          <z>
+            <noise type="gaussian">
+              <mean>0.0</mean>
+              <stddev>1.7e-2</stddev>
+              <bias_mean>0.1</bias_mean>
+              <bias_stddev>0.001</bias_stddev>
+            </noise>
+          </z>
+        </linear_acceleration>
+      </imu>
+    </sensor>
   </gazebo>
 </robot>

File: src/Anton_description/urdf/xacro/laser.xacro (robot description, xacro)
@@ -1,28 +1,27 @@
 <?xml version="1.0"?>
 <robot name="Anton" xmlns:xacro="http://www.ros.org/wiki/xacro">
-  <xacro:property name="laser_size_x" value="0.03"/>
-  <xacro:property name="laser_size_y" value="0.03"/>
-  <xacro:property name="laser_size_z" value="0.04"/>
-  <xacro:property name="laser_origin_x" value="0.065"/>
-  <xacro:property name="laser_origin_y" value="0"/>
-  <xacro:property name="laser_origin_z" value="0.035"/>
-  <link name="sensor_laser">
-    <visual>
+  <link name="lidar_link">
+    <inertial>
+      <origin xyz="0 0 0" rpy="0 0 0"/>
+      <mass value="0.125"/>
+      <inertia ixx="0.001"  ixy="0"  ixz="0" iyy="0.001" iyz="0" izz="0.001" />
+    </inertial>
+    <collision>
+      <origin xyz="0 0 0" rpy="0 0 0"/>
       <geometry>
-        <box size="${laser_size_x} ${laser_size_y} ${laser_size_z}"/>
-      </geometry>
-      <material name="blue"/>
-    </visual>
-    <collision>
-      <geometry>
-        <box size="${laser_size_x} ${laser_size_y} ${laser_size_z}"/>
+        <cylinder radius="0.0508" length="0.055"/>
       </geometry>
     </collision>
-    <xacro:box_inertia m="0.2" w="${laser_size_x}" h="${laser_size_y}" d="${laser_size_z}"/>
+    <visual>
+      <origin xyz="0 0 0" rpy="0 0 0"/>
+      <geometry>
+        <cylinder radius="0.0508" length="0.055"/>
+      </geometry>
+    </visual>
   </link>
-  <joint name="sensor_laser_joint" type="fixed">
-    <origin xyz="${laser_origin_x} ${laser_origin_y} ${laser_origin_z}" rpy="0 0 0" />
+  <joint name="lidar_joint" type="fixed">
     <parent link="base_link"/>
-    <child link="sensor_laser" />
+    <child link="lidar_link"/>
+    <origin xyz="0 0 0.12" rpy="0 0 0"/>
   </joint>
 </robot>

File: src/Anton_description/urdf/xacro/laserPlugin.xacro (robot description, xacro)
@@ -1,36 +1,37 @@
 <?xml version="1.0"?>
 <robot name="Anton" xmlns:xacro="http://www.ros.org/wiki/xacro">
-    <!--Gazebo Hokuyo Laser Plugin-->
-  <gazebo reference="sensor_laser">
-      <sensor type="ray" name="head_hokuyo_sensor">
-          <pose>0 0 0 0 0 0</pose>
-          <visualize>true</visualize>
-          <update_rate>20</update_rate>
-          <ray>
-              <scan>
-                  <horizontal>
-                      <samples>1440</samples>
-                      <resolution>1</resolution>
-                      <min_angle>-3.14159</min_angle>
-                      <max_angle>3.14159</max_angle>
-              </horizontal>
-          </scan>
-          <range>
-              <min>0.10</min>
-              <max>30.0</max>
-              <resolution>0.01</resolution>
-          </range>
-          <noise>
-              <type>gaussian</type>
-              <mean>0.0</mean>
-              <stddev>0.01</stddev>
-          </noise>
-      </ray>
-      <plugin name="gazebo_ros_head_hokuyo_controller" filename="libgazebo_ros_laser.so">
-          <topicName>/ai_rover_remastered/laser_scan/scan
-  </topicName>
-          <frameName>sensor_laser</frameName>
-      </plugin>
-      </sensor>
-  </gazebo>
+    <gazebo reference="lidar_link">
+        <sensor name="lidar" type="ray">
+            <always_on>true</always_on>
+            <visualize>true</visualize>
+            <update_rate>5</update_rate>
+            <ray>
+            <scan>
+                <horizontal>
+                <samples>360</samples>
+                <resolution>1.000000</resolution>
+                <min_angle>0.000000</min_angle>
+                <max_angle>6.280000</max_angle>
+                </horizontal>
+            </scan>
+            <range>
+                <min>0.120000</min>
+                <max>3.5</max>
+                <resolution>0.015000</resolution>
+            </range>
+            <noise>
+                <type>gaussian</type>
+                <mean>0.0</mean>
+                <stddev>0.01</stddev>
+            </noise>
+            </ray>
+            <plugin name="scan" filename="libgazebo_ros_ray_sensor.so">
+            <ros>
+                <remapping>~/out:=scan</remapping>
+            </ros>
+            <output_type>sensor_msgs/LaserScan</output_type>
+            <frame_name>lidar_link</frame_name>
+            </plugin>
+        </sensor>
+    </gazebo>
 </robot>

File: src/Anton_description/urdf/xacro/visuals.xacro (robot description, xacro)
@@ -5,8 +5,8 @@
     <material>Gazebo/Orange</material>
   </gazebo>
-  <gazebo reference="left_wheel">
+  <gazebo reference="drivewhl_l_link">
     <material>Gazebo/Blue</material>
   </gazebo>
-  <gazebo reference="right_wheel">
+  <gazebo reference="drivewhl_r_link">
     <material>Gazebo/Blue</material>
   </gazebo>

File: src/Anton_description/urdf/xacro/wheels.xacro (robot description, xacro)
@@ -1,33 +1,46 @@
 <?xml version="1.0"?>
 <robot name="Anton" xmlns:xacro="http://www.ros.org/wiki/xacro">
-<xacro:macro name="cylinder_inertia" params="m r h">
-  <inertial>
-    <mass value="${m}"/>
-    <inertia ixx="${m*(3*r*r+h*h)/12}" ixy="0" ixz="0" iyy="${m*(3*r*r+h*h)/12}" iyz="0" izz="${m*r*r/2}"/>
-  </inertial>
-</xacro:macro>
-<xacro:macro name="wheel" params="prefix reflect">
-  <link name="${prefix}_wheel">
-    <visual>
-      <origin xyz="0 0 0" rpy="${pi/2} 0 0"/>
-      <geometry>
-        <cylinder radius="${wheel_radius}" length="0.005"/>
-      </geometry>
-      <material name="blue"/>
-    </visual>
-    <collision>
-      <origin xyz="0 0 0" rpy="${pi/2} 0 0"/>
-      <geometry>
-        <cylinder radius="${wheel_radius}" length="0.005"/>
-      </geometry>
-    </collision>
-    <xacro:cylinder_inertia m="10" r="${wheel_radius}" h="0.005"/>
-  </link>
-  <joint name="${prefix}_wheel_joint" type="continuous">
-    <axis xyz="0 1 0" rpy="0 0 0" />
-    <parent link="base_link"/>
-    <child link="${prefix}_wheel"/>
-    <origin xyz="${wheel_joint_offset} ${((base_width/2)+base_wheel_gap)*reflect} -0.005" rpy="0 0 0"/>
-  </joint>
-</xacro:macro>
+  <xacro:macro name="cylinder_inertia" params="m r h">
+      <inertial>
+        <origin xyz="0 0 0" rpy="${pi/2} 0 0" />
+        <mass value="${m}"/>
+        <inertia ixx="${(m/12) * (3*r*r + h*h)}" ixy = "0" ixz = "0" iyy="${(m/12) * (3*r*r + h*h)}" iyz = "0" izz="${(m/2) * (r*r)}"/>
+      </inertial>
+  </xacro:macro>
+  <xacro:macro name="wheel" params="prefix x_reflect y_reflect">
+    <link name="${prefix}_link">
+      <visual>
+        <origin xyz="0 0 0" rpy="${pi/2} 0 0"/>
+        <geometry>
+            <cylinder radius="${wheel_radius}" length="${wheel_width}"/>
+        </geometry>
+        <material name="Gray">
+          <color rgba="0.5 0.5 0.5 1.0"/>
+        </material>
+      </visual>
+      <collision>
+        <origin xyz="0 0 0" rpy="${pi/2} 0 0"/>
+        <geometry>
+          <cylinder radius="${wheel_radius}" length="${wheel_width}"/>
+        </geometry>
+        <surface>
+        <friction>
+          <ode>
+            <mu>0.05</mu>
+            <mu2>0.05</mu2>
+          </ode>
+        </friction>
+      </surface>
+      </collision>
+      <xacro:cylinder_inertia m="5" r="${wheel_radius}" h="${wheel_width}"/>
+    </link>
+    <joint name="${prefix}_joint" type="continuous">
+      <parent link="base_link"/>
+      <child link="${prefix}_link"/>
+      <origin xyz="${x_reflect*wheel_xoff} ${y_reflect*(base_width/2+wheel_ygap)} ${-wheel_zoff}" rpy="0 0 0"/>
+      <axis xyz="0 1 0"/>
+    </joint>
+  </xacro:macro>
+  <xacro:wheel prefix="drivewhl_l" x_reflect="-1" y_reflect="1" />
+  <xacro:wheel prefix="drivewhl_r" x_reflect="-1" y_reflect="-1" />
 </robot>
